Commit message: Changed center_laser to OS1 Simulation: https://gitlab.laas.fr/gepetto/ouster-gazebo-simulation Changed FOV and resolution of front camera

File: prius_description/urdf/prius.urdf (robot description, URDF)
Before this commit: robot prius, 28 links, 27 joints
Joints:
- joint front_camera_joint: origin xyz=0 -0.4 1.4 rpy=0 0.05 -1.5707 -> xyz=0 -0.9 1.1 rpy=0 0 -1.5707

Commit message: Initial ros2 commit

File: prius_description/urdf/prius.urdf (robot description, URDF)
Before this commit: robot prius, 28 links, 27 joints
Joints:
- joint front_left_laser_joint: origin xyz=1 -2.3 0.5 rpy=0 0.05 0 -> xyz=1 -1.9 0.5 rpy=0 0.05 0
- joint front_right_laser_joint: origin xyz=-1 -2.3 0.5 rpy=0 0.05 3.14 -> xyz=-1 -1.9 0.5 rpy=0 0.05 3.14
